File: radio-module.kicad_pcb (KiCad board)
At the start: 4 copper layers, 80.2 x 22.1 mm, 154 parts, among them J1 MM8130-2600RA2, J2 2X05, J3 M.2-M+B-Pins, SW1 PTS840_GK_SMTR_LFS, SW2 PTS840_GK_SMTR_LFS, U1 UPD720202, U2 SST25VF512A, U3 CoralAccelerator, U4 NRF52840, U5 TPS61232DRCR, U6 NCP380HMUAJAATBG, U7 TLV62568PDRLT, U8 BME280, Y1 NX3225SA-24M, Y2 ABM11W-101-32.0000MHZ-T3, Y3 ABS06-32.768KHZ-9-1-T

Commit message: Cleanup
Parts:
- ANT1: footprint antmicro-pcie-radio-module-footprints:Linx-ANT-2.45-CHP-T-MFG -> radio-module-footprints:Linx-ANT-2.45-CHP-T-MFG
- C1, C10, C11, C12, C13, C14, C15, C16, C17, C18, C19, C2, C20, C21, C22, C23, C24, C25, C26, C27, C28, C29, C3, C31, C32, C33, C34, C35, C36, C37, C38, C39, C4, C40, C41, C42, C43, C44, C45, C46, C47, C48, C49, C5, C50, C51, C52, C53, C54, C55, C56, C57, C59, C6, C62, C65, C67, C68, C69, C7, C70, C71, C9: footprint antmicro-pcie-radio-module-footprints:0402-cap -> radio-module-footprints:0402-cap
- C30, C60, C63, C66, C8: footprint antmicro-pcie-radio-module-footprints:0805-cap -> radio-module-footprints:0805-cap
- C58, C61, C64: footprint antmicro-pcie-radio-module-footprints:Panasonic_Electronic_Components-CD-0-0-MFG -> radio-module-footprints:Panasonic_Electronic_Components-CD-0-0-MFG
- D1, D3, D4: footprint antmicro-pcie-radio-module-footprints:LED0603 -> radio-module-footprints:LED0603
- D2: footprint antmicro-pcie-radio-module-footprints:LED_APHF1608LSEEQBDZGKC -> radio-module-footprints:LED_APHF1608LSEEQBDZGKC
- FB1, R39: footprint antmicro-pcie-radio-module-footprints:0805-res -> radio-module-footprints:0805-res
- J1: footprint antmicro-pcie-radio-module-footprints:Murata-MM8130-2600RA2-MFG -> radio-module-footprints:Murata-MM8130-2600RA2-MFG
- J2: footprint antmicro-pcie-radio-module-footprints:ARM_SWD -> radio-module-footprints:ARM_SWD
- J3: footprint antmicro-pcie-radio-module-footprints:M.2-M+B-Keys -> radio-module-footprints:M.2-M+B-Keys
- L1, L2: footprint antmicro-pcie-radio-module-footprints:0603-res -> radio-module-footprints:0603-res
- L3, L4, R1, R10, R11, R12, R13, R14, R15, R16, R17, R18, R19, R2, R20, R21, R22, R23, R24, R25, R26, R27, R28, R29, R3, R30, R31, R32, R33, R34, R35, R36, R37, R38, R4, R40, R41, R5, R6, R7, R8, R9: footprint antmicro-pcie-radio-module-footprints:0402-res -> radio-module-footprints:0402-res
- L5: footprint antmicro-pcie-radio-module-footprints:Coilcraft-XFL4020-0-0-MFG -> radio-module-footprints:Coilcraft-XFL4020-0-0-MFG
- L6: footprint antmicro-pcie-radio-module-footprints:Murata-DFE201610C-0-0-IPC_B -> radio-module-footprints:Murata-DFE201610C-0-0-IPC_B
- MP1: footprint antmicro-pcie-radio-module-footprints:M.2-Stud -> radio-module-footprints:M.2-Stud
- N1: footprint antmicro-pcie-radio-module-footprints:antmicro-logo_scaled_12mm -> radio-module-footprints:antmicro-logo_scaled_12mm
- N2: footprint antmicro-pcie-radio-module-footprints:OSHW-Logo2_7.3x6mm_Copper_Mask -> radio-module-footprints:OSHW-Logo2_7.3x6mm_Copper_Mask
- SW1, SW2: footprint antmicro-pcie-radio-module-footprints:CK-PTS840_GK_SMTR_LFS-0 -> radio-module-footprints:CK-PTS840_GK_SMTR_LFS-0
- TP11, TP12, TP16, TP17, TP18, TP19, TP23, TP25, TP26, TP27, TP28: footprint antmicro-pcie-radio-module-footprints:Testpoint_smd_1mm -> radio-module-footprints:Testpoint_smd_1mm
- U1: footprint antmicro-pcie-radio-module-footprints:QFN48-Renesas-UPD720202 -> radio-module-footprints:QFN48-Renesas-UPD720202
- U2: footprint antmicro-pcie-radio-module-footprints:SOIC8-SST25VF512A-33-4I-SAE-Level_B -> radio-module-footprints:SOIC8-SST25VF512A-33-4I-SAE-Level_B
- U3: footprint antmicro-pcie-radio-module-footprints:MODULE_G313-06329-00 -> radio-module-footprints:MODULE_G313-06329-00
- U4: footprint antmicro-pcie-radio-module-footprints:Nordic_Semiconductor-NRF52840-QIAA-R-0-0-MFG -> radio-module-footprints:Nordic_Semiconductor-NRF52840-QIAA-R-0-0-MFG
- U5: footprint antmicro-pcie-radio-module-footprints:VSON-10-1EP_3x3mm -> radio-module-footprints:VSON-10-1EP_3x3mm
- U6: footprint antmicro-pcie-radio-module-footprints:ON_Semiconductor-517AB-04_2013-C-IPC_B -> radio-module-footprints:ON_Semiconductor-517AB-04_2013-C-IPC_B
- U7: footprint antmicro-pcie-radio-module-footprints:SOT-563 -> radio-module-footprints:SOT-563
- U8: footprint antmicro-footprints:Pressure_Sensor_LGA-8_2.5x2.5mm_BME280 -> radio-module-footprints:Pressure_Sensor_LGA-8_2.5x2.5mm_BME280
- Y1: footprint antmicro-pcie-radio-module-footprints:NDK-NX3225SA-0-0-MFG -> radio-module-footprints:NDK-NX3225SA-0-0-MFG
- Y2: footprint antmicro-pcie-radio-module-footprints:Abracon-ABM11W-0-0-0 -> radio-module-footprints:Abracon-ABM11W-0-0-0
- Y3: footprint antmicro-pcie-radio-module-footprints:Abracon-ABS06-32.768KHZ-T-0 -> radio-module-footprints:Abracon-ABS06-32.768KHZ-T-0
