File: nRF52840.kicad_sch (KiCad schematic)
At the start: 55 parts, among them J1 MM8130-2600RA2, J2 2X05, SW1 PTS840_GK_SMTR_LFS, U4 NRF52840, U8 BME280, Y2 ABM11W-101-32.0000MHZ-T3, Y3 ABS06-32.768KHZ-9-1-T

Commit message: Loclib
Parts:
- R53: footprint antmicro-footprints:0402-res -> m2-smart-iot-module-footprints:0402-res; symbol antmicroResistors0402:R_1k_0402 -> m2-smart-iot-module:R_1k_0402
