File: powerSupply.kicad_sch (KiCad schematic)
At the start: 41 parts, among them SW2 PTS840_GK_SMTR_LFS, U10 MIC2877-5.0YFT-TR, U6 AP22652W6-7, U9 NCP1599MNTWG

Commit message: Loclib
Parts:
- R33: footprint antmicro-footprints:0402-res -> m2-smart-iot-module-footprints:0402-res; symbol antmicroResistors0402:R_200k_0402 -> m2-smart-iot-module:R_200k_0402
- R54: footprint antmicro-footprints:0402-res -> m2-smart-iot-module-footprints:0402-res; symbol antmicroResistors0402:R_1k_0402 -> m2-smart-iot-module:R_1k_0402
- R62: footprint antmicro-footprints:0402-res -> m2-smart-iot-module-footprints:0402-res; symbol antmicroResistors0402:R_10k_0402 -> m2-smart-iot-module:R_10k_0402
