File: powerSupply.kicad_sch (KiCad schematic)
At the start: 41 parts, among them SW2 PTS840_GK_SMTR_LFS, U10 MIC2877-5.0YFT-TR, U6 AP22652W6-7, U9 NCP1599MNTWG

Commit message: [#102286] Fix legacy DNP
Parts:
- R39, SW2: DNP DNP -> (none); now not fitted
Changed lines of the file:
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@@
 		(on_board yes)
 		(in_pos_files yes)
-		(dnp no)
+		(dnp yes)
 		(property "Reference" "R39"
 			(at 280.67 37.338 0)
@@
 			)
 		)
-		(property "DNP" "DNP"
-			(at 280.67 42.1386 0)
-			(show_name no)
-			(do_not_autoplace no)
-			(effects
-				(font
-					(size 1.27 1.27)
-				)
-			)
-		)
 		(pin "1"
 		)
@@
 		(on_board yes)
 		(in_pos_files yes)
-		(dnp no)
+		(dnp yes)
 		(property "Reference" "SW2"
 			(at 66.675 160.02 0)
@@
 			(hide yes)
 			(show_name no)
-			(do_not_autoplace no)
-			(effects
-				(font
-					(size 1.27 1.27)
-				)
-			)
-		)
-		(property "DNP" "DNP"
-			(at 69.85 160.655 0)
-			(hide yes)
-			(show_name no)
