File: m2-smart-iot-module.kicad_sch (KiCad schematic)
At the start: 3 parts

Commit message: [#102286] Set exclude from BOM & pnp for MP1
Parts:
- MP1: now left out of the parts list
Changed lines of the file:
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@@
 		(body_style 1)
 		(exclude_from_sim no)
-		(in_bom yes)
+		(in_bom no)
 		(on_board yes)
-		(in_pos_files yes)
+		(in_pos_files no)
 		(dnp no)
 		(property "Reference" "MP1"
