File: coralAccelerator.kicad_sch (KiCad schematic)
At the start: 22 parts, among them Q1 BSS123, U3 CoralAccelerator, U5 AP2120N-1.8TRG1, U7 TLV803EF29DBZR

Commit message: [#102286] Fix legacy DNP
Parts:
- R37, R45, R46: DNP DNP -> (none); now not fitted
Changed lines of the file:
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@@
 		(on_board yes)
 		(in_pos_files yes)
-		(dnp no)
+		(dnp yes)
 		(property "Reference" "R37"
 			(at 68.58 75.565 0)
@@
 		(property "Val" "8k2"
 			(at 78.74 75.565 0)
-			(show_name no)
-			(do_not_autoplace no)
-			(effects
-				(font
-					(size 1.27 1.27)
-				)
-			)
-		)
-		(property "DNP" "DNP"
-			(at 73.66 76.835 0)
 			(show_name no)
 			(do_not_autoplace no)
@@
 		(on_board yes)
 		(in_pos_files yes)
-		(dnp no)
+		(dnp yes)
 		(property "Reference" "R45"
 			(at 153.035 80.01 0)
@@
 		(property "Val" "0R"
 			(at 153.035 81.915 0)
-			(show_name no)
-			(do_not_autoplace no)
-			(effects
-				(font
-					(size 1.27 1.27)
-				)
-			)
-		)
-		(property "DNP" "DNP"
-			(at 153.035 84.455 0)
 			(show_name no)
 			(do_not_autoplace no)
@@
 		(on_board yes)
 		(in_pos_files yes)
-		(dnp no)
+		(dnp yes)
 		(property "Reference" "R46"
 			(at 153.035 89.535 0)
@@
 			(show_name no)
 			(do_not_autoplace no)
-			(effects
-				(font
-					(size 1.27 1.27)
-				)
-			)
-		)
-		(property "DNP" "DNP"
-			(at 153.035 86.995 0)
-			(show_name no)
-			(do_not_autoplace no)

Commit message: [#102286] Unify C_100n_0402 capacitors to use single MPN
Refs: C1, C3, C6, C7, C10, C13, C17, C18, C25-C29, C33, C36, C39, C41,
C44, C67-C71

Change from 0402X104K6R3CT to GRM155R61H104KE14D (same but limit 50V
instead of 6V3)
Parts:
- C28, C29, C67, C68, C69: MPN 0402X104K6R3CT -> GRM155R61H104KE14D; Manufacturer Walsin -> Murata
Changed lines of the file:
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@@
 		)
 		(property "Intersheetrefs" "${INTERSHEET_REFS}"
-			(at 0 0 0)
-			(hide yes)
-			(show_name no)
-			(do_not_autoplace no)
-			(effects
-				(font
-					(size 1.27 1.27)
-				)
+			(at 90.1069 165.1 0)
+			(hide yes)
+			(show_name no)
+			(do_not_autoplace no)
+			(effects
+				(font
+					(size 1.27 1.27)
+				)
+				(justify right)
 			)
 		)
@@
 		)
 		(property "Intersheetrefs" "${INTERSHEET_REFS}"
-			(at 0 0 0)
-			(hide yes)
-			(show_name no)
-			(do_not_autoplace no)
-			(effects
-				(font
-					(size 1.27 1.27)
-				)
+			(at 153.035 33.5616 90)
+			(hide yes)
+			(show_name no)
+			(do_not_autoplace no)
+			(effects
+				(font
+					(size 1.27 1.27)
+				)
+				(justify left)
 			)
 		)
@@
 		)
 		(property "Intersheetrefs" "${INTERSHEET_REFS}"
-			(at 0 0 0)
-			(hide yes)
-			(show_name no)
-			(do_not_autoplace no)
-			(effects
-				(font
-					(size 1.27 1.27)
-				)
+			(at 41.8166 241.3 0)
+			(hide yes)
+			(show_name no)
+			(do_not_autoplace no)
+			(effects
+				(font
+					(size 1.27 1.27)
+				)
+				(justify right)
 			)
 		)
@@
 		)
 		(property "Intersheetrefs" "${INTERSHEET_REFS}"
-			(at 0 0 0)
-			(hide yes)
-			(show_name no)
-			(do_not_autoplace no)
-			(effects
-				(font
-					(size 1.27 1.27)
-				)
+			(at 47.8491 84.455 0)
+			(hide yes)
+			(show_name no)
+			(do_not_autoplace no)
+			(effects
+				(font
+					(size 1.27 1.27)
+				)
+				(justify right)
 			)
 		)
@@
 		)
 		(property "Intersheetrefs" "${INTERSHEET_REFS}"
-			(at 0 0 0)
-			(hide yes)
-			(show_name no)
-			(do_not_autoplace no)
-			(effects
-				(font
-					(size 1.27 1.27)
-				)
+			(at 66.5816 48.26 0)
+			(hide yes)
+			(show_name no)
+			(do_not_autoplace no)
+			(effects
+				(font
+					(size 1.27 1.27)
+				)
+				(justify right)
 			)
 		)
@@
 		)
 		(property "Intersheetrefs" "${INTERSHEET_REFS}"
-			(at 0 0 0)
-			(hide yes)
-			(show_name no)
-			(do_not_autoplace no)
-			(effects
-				(font
-					(size 1.27 1.27)
-				)
+			(at 52.6116 200.025 0)
+			(hide yes)
+			(show_name no)
+			(do_not_autoplace no)
+			(effects
+				(font
+					(size 1.27 1.27)
+				)
+				(justify right)
 			)
 		)
@@
 		)
 		(property "Intersheetrefs" "${INTERSHEET_REFS}"
-			(at 0 0 0)
-			(hide yes)
-			(show_name no)
-			(do_not_autoplace no)
-			(effects
-				(font
-					(size 1.27 1.27)
-				)
+			(at 47.7886 86.995 0)
+			(hide yes)
+			(show_name no)
+			(do_not_autoplace no)
+			(effects
+				(font
+					(size 1.27 1.27)
+				)
+				(justify right)
 			)
 		)
@@
 		)
 		(property "Intersheetrefs" "${INTERSHEET_REFS}"
-			(at 0 0 0)
-			(hide yes)
-			(show_name no)
-			(do_not_autoplace no)
-			(effects
-				(font
-					(size 1.27 1.27)
-				)
+			(at 41.6957 76.835 0)
+			(hide yes)
+			(show_name no)
+			(do_not_autoplace no)
+			(effects
+				(font
+					(size 1.27 1.27)
+				)
+				(justify right)
 			)
 		)
@@
 		)
 		(property "Intersheetrefs" "${INTERSHEET_REFS}"
-			(at 0 0 0)
-			(hide yes)
-			(show_name no)
-			(do_not_autoplace no)
-			(effects
-				(font
-					(size 1.27 1.27)
-				)
+			(at 177.077 69.215 0)
+			(hide yes)
+			(show_name no)
+			(do_not_autoplace no)
+			(effects
+				(font
+					(size 1.27 1.27)
+				)
+				(justify left)
 			)
 		)
@@
 			)
 		)
-		(property "Manufacturer" "Walsin"
+		(property "Manufacturer" "Murata"
 			(at 80.01 240.03 0)
 			(hide yes)
@@
 			)
 		)
-		(property "MPN" "0402X104K6R3CT"
+		(property "MPN" "GRM155R61H104KE14D"
 			(at 80.01 242.57 0)
 			(hide yes)
@@
 			)
 		)
-		(property "Manufacturer" "Walsin"
+		(property "Manufacturer" "Murata"
 			(at 67.31 240.03 0)
 			(hide yes)
@@
 			)
 		)
-		(property "MPN" "0402X104K6R3CT"
+		(property "MPN" "GRM155R61H104KE14D"
 			(at 67.31 242.57 0)
 			(hide yes)
@@
 			)
 		)
-		(property "Manufacturer" "Walsin"
+		(property "Manufacturer" "Murata"
 			(at 95.885 82.55 0)
 			(hide yes)
@@
 			)
 		)
-		(property "MPN" "0402X104K6R3CT"
+		(property "MPN" "GRM155R61H104KE14D"
 			(at 95.885 85.09 0)
 			(hide yes)
@@
 			)
 		)
-		(property "Manufacturer" "Walsin"
+		(property "Manufacturer" "Murata"
 			(at 102.87 240.03 0)
 			(hide yes)
@@
 			)
 		)
-		(property "MPN" "0402X104K6R3CT"
+		(property "MPN" "GRM155R61H104KE14D"
 			(at 102.87 242.57 0)
 			(hide yes)
@@
 			)
 		)
-		(property "Manufacturer" "Walsin"
+		(property "Manufacturer" "Murata"
 			(at 115.57 240.03 0)
 			(hide yes)
@@
 			)
 		)
-		(property "MPN" "0402X104K6R3CT"
+		(property "MPN" "GRM155R61H104KE14D"
 			(at 115.57 242.57 0)
 			(hide yes)
