File: pcie-usb-bridge.kicad_sch (KiCad schematic)
At the start: 58 parts, among them IC1 UPD720201K8-711-BAC-A, U2 SST25VF512A, Y1 NX3225SA-24M

Commit message: [#102286] Bump to KiCad10
Parts:
- R47, R48: value ~ -> (none)

Commit message: [#102286] Fix legacy DNP
Parts:
- R11, R8: DNP DNP -> (none); now not fitted
Changed lines of the file:
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@@
 		(on_board yes)
 		(in_pos_files yes)
-		(dnp no)
+		(dnp yes)
 		(property "Reference" "R8"
 			(at 194.818 57.277 90)
@@
 				)
 				(justify left)
-			)
-		)
-		(property "DNP" "DNP"
-			(at 196.85 54.61 90)
-			(show_name no)
-			(do_not_autoplace no)
-			(effects
-				(font
-					(size 1.27 1.27)
-				)
 			)
 		)
@@
 		(on_board yes)
 		(in_pos_files yes)
-		(dnp no)
+		(dnp yes)
 		(property "Reference" "R11"
 			(at 208.788 57.277 90)
@@
 			)
 		)
-		(property "DNP" "DNP"
-			(at 210.82 54.61 90)
-			(show_name no)
-			(do_not_autoplace no)
-			(effects
-				(font
-					(size 1.27 1.27)
-				)
-			)
-		)

Commit message: [#102286] Unify C_100n_0402 capacitors to use single MPN
Refs: C1, C3, C6, C7, C10, C13, C17, C18, C25-C29, C33, C36, C39, C41,
C44, C67-C71

Change from 0402X104K6R3CT to GRM155R61H104KE14D (same but limit 50V
instead of 6V3)
Parts:
- C1, C10, C13, C17, C18, C25, C26, C27, C3, C6, C7: MPN 0402X104K6R3CT -> GRM155R61H104KE14D; Manufacturer Walsin -> Murata
Changed lines of the file:
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@@
 		)
 		(property "Intersheetrefs" "${INTERSHEET_REFS}"
-			(at 0 0 0)
+			(at 175.1364 31.75 0)
 			(hide yes)
 			(show_name no)
@@
 					(size 1.27 1.27)
 				)
+				(justify right)
 			)
 		)
@@
 		)
 		(property "Intersheetrefs" "${INTERSHEET_REFS}"
-			(at 0 0 0)
+			(at 272.5386 46.99 0)
 			(hide yes)
 			(show_name no)
@@
 					(size 1.27 1.27)
 				)
+				(justify left)
 			)
 		)
@@
 		)
 		(property "Intersheetrefs" "${INTERSHEET_REFS}"
-			(at 0 0 0)
+			(at 251.5836 44.45 0)
 			(hide yes)
 			(show_name no)
@@
 					(size 1.27 1.27)
 				)
+				(justify left)
 			)
 		)
@@
 			)
 		)
-		(property "Manufacturer" "Walsin"
+		(property "Manufacturer" "Murata"
 			(at 180.34 137.16 0)
 			(hide yes)
@@
 			)
 		)
-		(property "MPN" "0402X104K6R3CT"
+		(property "MPN" "GRM155R61H104KE14D"
 			(at 180.34 139.7 0)
 			(hide yes)
@@
 			)
 		)
-		(property "Manufacturer" "Walsin"
+		(property "Manufacturer" "Murata"
 			(at 193.04 137.16 0)
 			(hide yes)
@@
 			)
 		)
-		(property "MPN" "0402X104K6R3CT"
+		(property "MPN" "GRM155R61H104KE14D"
 			(at 193.04 139.7 0)
 			(hide yes)
@@
 			)
 		)
-		(property "Manufacturer" "Walsin"
+		(property "Manufacturer" "Murata"
 			(at 107.315 163.195 0)
 			(hide yes)
@@
 			)
 		)
-		(property "MPN" "0402X104K6R3CT"
+		(property "MPN" "GRM155R61H104KE14D"
 			(at 107.315 165.735 0)
 			(hide yes)
@@
 			)
 		)
-		(property "Manufacturer" "Walsin"
+		(property "Manufacturer" "Murata"
 			(at 128.27 163.195 0)
 			(hide yes)
@@
 			)
 		)
-		(property "MPN" "0402X104K6R3CT"
+		(property "MPN" "GRM155R61H104KE14D"
 			(at 128.27 165.735 0)
 			(hide yes)
@@
 			)
 		)
-		(property "Manufacturer" "Walsin"
+		(property "Manufacturer" "Murata"
 			(at 92.075 163.195 0)
 			(hide yes)
@@
 			)
 		)
-		(property "MPN" "0402X104K6R3CT"
+		(property "MPN" "GRM155R61H104KE14D"
 			(at 92.075 165.735 0)
 			(hide yes)
@@
 			)
 		)
-		(property "Manufacturer" "Walsin"
+		(property "Manufacturer" "Murata"
 			(at 148.59 163.195 0)
 			(hide yes)
@@
 			)
 		)
-		(property "MPN" "0402X104K6R3CT"
+		(property "MPN" "GRM155R61H104KE14D"
 			(at 148.59 165.735 0)
 			(hide yes)
@@
 			)
 		)
-		(property "Manufacturer" "Walsin"
+		(property "Manufacturer" "Murata"
 			(at 45.085 163.83 0)
 			(hide yes)
@@
 			)
 		)
-		(property "MPN" "0402X104K6R3CT"
+		(property "MPN" "GRM155R61H104KE14D"
 			(at 45.085 166.37 0)
 			(hide yes)
@@
 			)
 		)
-		(property "Manufacturer" "Walsin"
+		(property "Manufacturer" "Murata"
 			(at 38.1 163.83 0)
 			(hide yes)
@@
 			)
 		)
-		(property "MPN" "0402X104K6R3CT"
+		(property "MPN" "GRM155R61H104KE14D"
 			(at 38.1 166.37 0)
 			(hide yes)
@@
 			)
 		)
-		(property "Manufacturer" "Walsin"
+		(property "Manufacturer" "Murata"
 			(at 64.77 109.22 0)
 			(hide yes)
@@
 			)
 		)
-		(property "MPN" "0402X104K6R3CT"
+		(property "MPN" "GRM155R61H104KE14D"
 			(at 62.23 109.22 0)
 			(hide yes)
@@
 			)
 		)
-		(property "Manufacturer" "Walsin"
+		(property "Manufacturer" "Murata"
 			(at 60.96 105.41 0)
 			(hide yes)
@@
 			)
 		)
-		(property "MPN" "0402X104K6R3CT"
+		(property "MPN" "GRM155R61H104KE14D"
 			(at 58.42 105.41 0)
 			(hide yes)
@@
 			)
 		)
-		(property "Manufacturer" "Walsin"
+		(property "Manufacturer" "Murata"
 			(at 246.38 45.085 0)
 			(hide yes)
@@
 			)
 		)
-		(property "MPN" "0402X104K6R3CT"
+		(property "MPN" "GRM155R61H104KE14D"
 			(at 246.38 47.625 0)
 			(hide yes)
