File: ftdi.kicad_sch (KiCad schematic)
At the start: 28 parts, among them U1 FT4232H-56Q, U11 93LC56CT-IMC, Y4 ABM8G-12M-18-D2Y-T

Commit message: [#102286] Set MPN & MFR in U11
Parts:
- U11: MPN (none) -> 93LC56CT-IMC; Manufacturer (none) -> Microchip Technology
Changed lines of the file:
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@@
+			)
+		)
+		(property "MPN" "93LC56CT-IMC"
+			(at 69.85 111.76 0)
+			(hide yes)
+			(show_name no)
+			(do_not_autoplace no)
+			(effects
+				(font
+					(size 1.27 1.27)
+				)
+			)
+		)
+		(property "Manufacturer" "Microchip Technology"
+			(at 69.85 111.76 0)
+			(hide yes)
+			(show_name no)
+			(do_not_autoplace no)
+			(effects
+				(font
+					(size 1.27 1.27)
+				)
 			)
 		)
